Commit message: 現在の状況をすべてコミット

File: src/sim/urdf/_d435.gazebo.xacro (robot description, xacro)
@@ -23,8 +23,11 @@
       <!--<max_vel>0.01</max_vel>
       <min_depth>0</min_depth>-->
+      <!-- colorの解像度をここで変える???????-->
       <sensor name="${camera_name}color" type="camera">
         <camera name="${camera_name}">
           <horizontal_fov>${69.4*deg_to_rad}</horizontal_fov>
           <image>
+            <!-- <width>1280</width>
+            <height>720</height> -->
             <width>640</width>
             <height>360</height>

File: src/sim/urdf/beego.urdf (robot description, URDF)
Before this commit: robot beego, 7 links, 6 joints
Joints:
- joint left_wheel_joint: type continuous -> fixed
- joint right_wheel_joint: type continuous -> fixed

File: src/sim/urdf/beego.urdf.xacro (robot description, xacro)
@@ -67,5 +67,5 @@
     </inertial>
   </link>
-  <joint name="right_wheel_joint" type="continuous">
+  <joint name="right_wheel_joint" type="fixed">
     <origin xyz="0.02225 -0.1308 -0.01" rpy="${-M_PI/2} 0 0"/>
     <parent link="base_link"/>
@@ -100,5 +100,5 @@
     </inertial>
   </link>
-  <joint name="left_wheel_joint" type="continuous">
+  <joint name="left_wheel_joint" type="fixed">
     <origin xyz="0.02225 0.1308 -0.01" rpy="${M_PI/2} 0 0"/>
     <parent link="base_link"/>
@@ -261,11 +261,11 @@
   <gazebo reference="base_link">
     <selfCollide>true</selfCollide>
-    <mu1 value="0.05"/>
-    <mu2 value="0.05"/>
+    <mu1 value="0.0"/>
+    <mu2 value="0.0"/>
   </gazebo>
   <gazebo reference="left_wheel_link">
     <selfCollide>true</selfCollide>
-    <mu1 value="1.0"/>
-    <mu2 value="1.0"/>
+    <mu1 value="0.0"/>
+    <mu2 value="0.0"/>
     <!--<kp value="10000000.0"/>
     <kd value="1.0"/>-->
@@ -273,6 +273,6 @@
   <gazebo reference="right_wheel_link">
     <selfCollide>true</selfCollide>
-    <mu1 value="1.0"/>
-    <mu2 value="1.0"/>
+    <mu1 value="0.0"/>
+    <mu2 value="0.0"/>
     <!--<kp value="10000000.0"/>
     <kd value="1.0"/>-->
@@ -280,6 +280,6 @@
   <gazebo reference="caster_link">
     <selfCollide>true</selfCollide>
-    <mu1 value="0.1"/>
-    <mu2 value="0.1"/>
+    <mu1 value="0.0"/>
+    <mu2 value="0.0"/>
   </gazebo>
   <!-- <xacro:arg name="use_nominal_extrinsics" default="false" />
@@ -288,6 +288,9 @@
     <origin xyz="0 0 0" rpy="0 0 0"/>
   </xacro:sensor_d435i> -->
+  <!-- 24deg / 0.418879rad:  -->
+  <!-- 23deg / 0.401426rad -->
+  <!-- 22.5deg /0.3926991 -->
   <xacro:sensor_d435 parent="base_footprint">
-    <origin rpy="0 0.418879 0" xyz="0.3 -${0.0175 + 0.015} 0.21"/>
+    <origin rpy="0 0.3926991 0" xyz="0.3 -${0.0175 + 0.015} 0.21"/>
   </xacro:sensor_d435>
 <!-- <gazebo reference="camera_link">
