Commit message: gazebo環境でpf回せるようにした

File: src/sim/urdf/beego.urdf (robot description, URDF)
Before this commit: robot beego, 7 links, 6 joints
Joints:
- joint camera_joint: origin xyz=0.3 0.0 0.21 rpy=0 0.3944444 0 -> xyz=0.3 0.0 0.21 rpy=0 0.436332 0

Commit message: pf用にロボットを動かせるようにした

File: src/sim/urdf/beego.urdf (robot description, URDF)
Before this commit: robot beego, 7 links, 6 joints
Links:
- link camera_link: geometry collision box size=0.1 0.1 0.1; visual box size=0.1 0.1 0.1
Joints:
- joint camera_joint: origin xyz=0.3 0.0 0.21 rpy=0 0.418879 0 -> xyz=0.3 0.0 0.21 rpy=0 0.3944444 0
- joint left_wheel_joint: type fixed -> continuous
- joint right_wheel_joint: type fixed -> continuous

File: src/sim/urdf/beego_old.urdf (robot description, URDF)
Before this commit: robot beego, 6 links, 5 joints
Links:
- added link camera_link; collision box size=0.1 0.1 0.1; visual box size=0.1 0.1 0.1
- link base_link: geometry collision box size=0.25 0.3 0.004; visual mesh filename=package://yamasemi_sim/meshes/base_link.STL
- link hokuyo_link: geometry collision box size=0.05 0.05 0.07; visual mesh filename=package://yamasemi_sim/meshes/hokuyo.dae
- link left_wheel_link: geometry collision cylinder length=${WHEEL_THICK} radius=${WHEEL_RAD}; visual mesh filename=package://yamasemi_sim/meshes/left_wheel_link.STL
- link right_wheel_link: geometry collision cylinder length=${WHEEL_THICK} radius=${WHEEL_RAD}; visual mesh filename=package://yamasemi_sim/meshes/right_wheel_link.STL
Joints:
- added joint camera_joint: type fixed, parent base_link, child camera_link, origin xyz=0 0.1 0 rpy=0 0.4 0, axis 0 1 0
