Commit message: gazebo環境に3つのカメラと地図を配置して同時にデータ取れるように改良

File: src/sim/urdf/_d435_chinpo.urdf.xacro (robot description, xacro)
@@ -1,15 +1,8 @@
 <?xml version="1.0"?>
-<!--
-License: Apache 2.0. See LICENSE file in root directory.
-Copyright(c) 2017 Intel Corporation. All Rights Reserved
-This is the URDF model for the Intel RealSense 430 camera, in it's
-aluminum peripherial evaluation case.
--->
-<!-- 別 -->
-<robot name="sensor_d435" xmlns:xacro="http://ros.org/wiki/xacro">
+<robot name="sensor_d435_chinpo" xmlns:xacro="http://ros.org/wiki/xacro">
   <!--File includes-->
   <xacro:include filename="$(find sim)/urdf/_d435.gazebo.xacro"/>
-  <xacro:macro name="sensor_d435" params="name:=camera
-    topics_ns:=camera
+  <xacro:macro name="sensor_d435_chinpo" params="name:=camera
+    topics_ns:=camera_chinpo
     parent *origin publish_pointcloud:=true">
     <xacro:property name="M_PI" value="3.1415926535897931" />

File: src/sim/urdf/beego.urdf.xacro (robot description, xacro)
@@ -13,7 +13,34 @@
   <xacro:arg name="use_nominal_extrinsics" default="false" />
   <xacro:include filename="$(find sim)/urdf/_d435.urdf.xacro"/>
+  <!-- <xacro:include filename="$(find sim)/urdf/_d435_chinpo.urdf.xacro"/> -->
   <material name="gray">
     <color rgba="0.75 0.75 0.75 1"/>
   </material>
+<!-- ロボットに追加のオブジェクトでカメラの重みで倒れないようにする -->
+  <link name="extra_weight">
+    <visual>
+      <origin xyz="0 0 0.15" rpy="0 0 0"/> <!-- 位置を調整 -->
+      <geometry>
+        <box size="0.1 0.1 0.1"/> <!-- サイズを設定 -->
+      </geometry>
+      <material name="gray"/>
+    </visual>
+    <collision>
+      <origin xyz="0 0 0.1" rpy="0 0 0"/>
+      <geometry>
+        <box size="0.1 0.1 0.1"/>
+      </geometry>
+    </collision>
+    <inertial>
+      <origin xyz="0 0 0.15" rpy="0 0 0"/>
+      <mass value="25.0"/> <!-- 重量を設定 -->
+      <inertia ixx="0.1" ixy="0" ixz="0" iyy="0.1" iyz="0" izz="0.1"/>
+    </inertial>
+  </link>
+  <joint name="extra_weight_joint" type="fixed">
+    <parent link="base_link"/>
+    <child link="extra_weight"/>
+    <origin xyz="0 0 0.1" rpy="0 0 0"/> <!-- 位置を調整 -->
+  </joint>
   <!-- ===============  Body =============== -->
   <link name="base_link">
@@ -301,6 +328,15 @@
   <!-- 23deg / 0.401426rad -->
   <!-- 22.5deg /0.3926991 -->
-  <xacro:sensor_d435 parent="base_footprint">
+  <!-- <xacro:sensor_d435_chinpo name="camera1" parent="base_footprint" topics_ns="camera1">
     <origin rpy="0 0.3926991 0" xyz="0.3 -${0.0175 + 0.015} 0.21"/>
+  </xacro:sensor_d435_chinpo> -->
+  <xacro:sensor_d435 name="camera1" parent="base_footprint" topics_ns="camera1">
+    <origin rpy="0 0.3926991 0" xyz="0.3 -${0.0175 + 0.015} 0.21"/>
+  </xacro:sensor_d435>
+  <xacro:sensor_d435 name="camera2" parent="base_footprint" topics_ns="camera2">
+    <origin rpy="0 0.3926991 0" xyz="0.3 -${0.0175 + 0.015} -0.79"/>
+  </xacro:sensor_d435>
+  <xacro:sensor_d435 name="camera3" parent="base_footprint" topics_ns="camera3">
+    <origin rpy="0 0.3926991 0" xyz="0.3 -${0.0175 + 0.015} -1.79"/>
   </xacro:sensor_d435>
 <!-- <gazebo reference="camera_link">
