Commit message: realsense-gazebo-pluginの導入

File: src/sim/urdf/beego.urdf.xacro (robot description, xacro)
@@ -11,4 +11,6 @@
   <xacro:property name="WHEEL_RAD" value="0.041"/>
   <xacro:property name="WHEEL_THICK" value="0.015"/>
+  <xacro:arg name="use_nominal_extrinsics" default="false" />
+  <xacro:include filename="$(find sim)/urdf/_d435.urdf.xacro"/>
   <material name="gray">
     <color rgba="0.75 0.75 0.75 1"/>
@@ -166,5 +168,5 @@
     </collision>
   </link> -->
-	<link name="camera_link">
+	<!-- <link name="camera_link">
 		<collision>
 			<origin xyz="0 0 0" rpy="0 0 0"/>
@@ -184,11 +186,12 @@
 			<inertia ixx="1e-6" ixy="0" ixz="0" iyy="1e-6" iyz="0" izz="1e-6" />
 		</inertial>
-	</link>
-	<joint name="camera_joint" type="fixed">
+	</link> -->
+  <!-- <link name="camera_link" /> -->
+	<!-- <joint name="camera_joint" type="fixed">
 		<parent link="base_link"/>
 		<child link="camera_link"/>
     <origin rpy="0 0.418879 0" xyz="0.3 0.0 0.21"/>
 		<axis xyz="0 1 0"/>
-	</joint>
+	</joint> -->
   <!-- ===============  Transmission =============== -->
   <transmission name="left_wheel_trans">
@@ -285,5 +288,8 @@
     <origin xyz="0 0 0" rpy="0 0 0"/>
   </xacro:sensor_d435i> -->
-<gazebo reference="camera_link">
+  <xacro:sensor_d435 parent="base_footprint">
+    <origin rpy="0 0.418879 0" xyz="0.3 -${0.0175 + 0.015} 0.21"/>
+  </xacro:sensor_d435>
+<!-- <gazebo reference="camera_link">
 		<sensor type="camera" name="camera1">
 			<update_rate>30.0</update_rate>
@@ -318,4 +324,4 @@
 			</plugin>
 		</sensor>
-	</gazebo>
+	</gazebo> -->
 </robot>

Commit message: 20240109の進捗

File: src/sim/urdf/beego.urdf.xacro (robot description, xacro)
@@ -18,9 +18,9 @@
   </material>
 <!-- ロボットに追加のオブジェクトでカメラの重みで倒れないようにする -->
-  <link name="extra_weight">
+  <!-- <link name="extra_weight">
     <visual>
-      <origin xyz="0 0 0.15" rpy="0 0 0"/> <!-- 位置を調整 -->
-      <geometry>
-        <box size="0.1 0.1 0.1"/> <!-- サイズを設定 -->
+      <origin xyz="0 0 0.15" rpy="0 0 0"/> 位置を調整
+      <geometry>
+        <box size="0.1 0.1 0.1"/> サイズを設定
       </geometry>
       <material name="gray"/>
@@ -34,5 +34,5 @@
     <inertial>
       <origin xyz="0 0 0.15" rpy="0 0 0"/>
-      <mass value="25.0"/> <!-- 重量を設定 -->
+      <mass value="25.0"/> 重量を設定
       <inertia ixx="0.1" ixy="0" ixz="0" iyy="0.1" iyz="0" izz="0.1"/>
     </inertial>
@@ -41,6 +41,6 @@
     <parent link="base_link"/>
     <child link="extra_weight"/>
-    <origin xyz="0 0 0.1" rpy="0 0 0"/> <!-- 位置を調整 -->
-  </joint>
+    <origin xyz="0 0 0.1" rpy="0 0 0"/> 位置を調整
+  </joint> -->
   <!-- ===============  Body =============== -->
   <link name="base_link">
@@ -334,10 +334,11 @@
     <origin rpy="0 0.3926991 0" xyz="0.3 -${0.0175 + 0.015} 0.21"/>
   </xacro:sensor_d435>
-  <xacro:sensor_d435 name="camera2" parent="base_footprint" topics_ns="camera2">
+  <!-- <xacro:sensor_d435 name="camera2" parent="base_footprint" topics_ns="camera2">
     <origin rpy="0 0.3926991 0" xyz="0.3 -${0.0175 + 0.015} -0.79"/>
   </xacro:sensor_d435>
-  <xacro:sensor_d435 name="camera3" parent="base_footprint" topics_ns="camera3">
+ -->
+  <!-- <xacro:sensor_d435 name="camera3" parent="base_footprint" topics_ns="camera3">
     <origin rpy="0 0.3926991 0" xyz="0.3 -${0.0175 + 0.015} -1.79"/>
-  </xacro:sensor_d435>
+  </xacro:sensor_d435> -->
 <!-- <gazebo reference="camera_link">
 		<sensor type="camera" name="camera1">

Commit message: 同時に実験出来るようにした

File: src/sim/urdf/beego.urdf.xacro (robot description, xacro)
@@ -18,9 +18,9 @@
   </material>
 <!-- ロボットに追加のオブジェクトでカメラの重みで倒れないようにする -->
-  <!-- <link name="extra_weight">
+  <link name="extra_weight">
     <visual>
-      <origin xyz="0 0 0.15" rpy="0 0 0"/> 位置を調整
-      <geometry>
-        <box size="0.1 0.1 0.1"/> サイズを設定
+      <origin xyz="0 0 0.15" rpy="0 0 0"/> //位置を調整
+      <geometry>
+        <box size="0.1 0.1 0.1"/> //サイズを設定
       </geometry>
       <material name="gray"/>
@@ -34,5 +34,5 @@
     <inertial>
       <origin xyz="0 0 0.15" rpy="0 0 0"/>
-      <mass value="25.0"/> 重量を設定
+      <mass value="25.0"/> // 重量を設定
       <inertia ixx="0.1" ixy="0" ixz="0" iyy="0.1" iyz="0" izz="0.1"/>
     </inertial>
@@ -41,6 +41,6 @@
     <parent link="base_link"/>
     <child link="extra_weight"/>
-    <origin xyz="0 0 0.1" rpy="0 0 0"/> 位置を調整
-  </joint> -->
+    <origin xyz="0 0 0.1" rpy="0 0 0"/> //位置を調整
+  </joint>
   <!-- ===============  Body =============== -->
   <link name="base_link">
@@ -334,11 +334,10 @@
     <origin rpy="0 0.3926991 0" xyz="0.3 -${0.0175 + 0.015} 0.21"/>
   </xacro:sensor_d435>
-  <!-- <xacro:sensor_d435 name="camera2" parent="base_footprint" topics_ns="camera2">
+  <xacro:sensor_d435 name="camera2" parent="base_footprint" topics_ns="camera2">
     <origin rpy="0 0.3926991 0" xyz="0.3 -${0.0175 + 0.015} -0.79"/>
   </xacro:sensor_d435>
- -->
-  <!-- <xacro:sensor_d435 name="camera3" parent="base_footprint" topics_ns="camera3">
+  <xacro:sensor_d435 name="camera3" parent="base_footprint" topics_ns="camera3">
     <origin rpy="0 0.3926991 0" xyz="0.3 -${0.0175 + 0.015} -1.79"/>
-  </xacro:sensor_d435> -->
+  </xacro:sensor_d435>
 <!-- <gazebo reference="camera_link">
 		<sensor type="camera" name="camera1">
